File: motor_controller_v1.kicad_pcb (KiCad board)
At the start: 2 copper layers, 17 parts, among them J1 Conn_01x01_Male, J2 Conn_01x01_Male, J3 Conn_01x10_Female, J4 Conn_01x01_Male, J5 Conn_01x01_Male, J6 Conn_01x01_Male, Q1 Q_NMOS_GDS, Q2 Q_NMOS_GDS, Q3 Q_NMOS_GDS, Q4 Q_NMOS_GDS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

Commit message: Finishing layout
Other:
- board outline added: 77.7 x 45.5 mm
